File: hardware/MCU.kicad_sch (KiCad schematic)
At the start: 0 parts

Commit message: feat：MCU最小系统原理图设计；SRAM原理图设计
Parts:
- added C1, C2: 10pF, Capacitor_SMD:C_0603_1608Metric, symbol Device:C
- added C10, C11, C13, C15, C16, C18, C19, C4, C5, C6, C7, C8, C9: 100nF, Capacitor_SMD:C_0603_1608Metric, symbol Device:C
- added C12, C14: 1uF, Capacitor_SMD:C_0603_1608Metric, symbol Device:C
- added C17, C3: 4.7uF, Capacitor_SMD:C_0603_1608Metric, symbol Device:C
- added J1: Conn_01x03_Pin, symbol Connector:Conn_01x03_Pin
- added R1, R2: 10kR, Resistor_SMD:R_0603_1608Metric, symbol Device:R
- added SW1: SW_MEC_5G, Button_Switch_SMD:SW_SPST_FSMSM, symbol Switch:SW_MEC_5G
- added U1: STM32G473QETxZ, Package_QFP:LQFP-128_14x14mm_P0.4mm, symbol MCU_ST_STM32G4:STM32G473QETx_by_fuc
- added U2: IS61W204816BLL, Package_SO:TSOP-I-48_18.4x12mm_P0.5mm, symbol Memory_RAM:IS61WV204816BLL-10TLI
- added Y1: 25MHz, Crystal:Crystal_SMD_3225-4Pin_3.2x2.5mm, symbol Device:Crystal_GND24
Connections:
- new net: U2.19 (NC), U2.6 (NC)
- new net: R1.1, U1.123 (PB8)
- new net +3.3V: C10.1, C11.1, C17.1, C18.1, C19.1, C3.1, C4.1, C5.1, C6.1, C7.1, C8.1, C9.1, R2.2, U1.111 (VDD), U1.128 (VDD), U1.13 (VDD), U1.31 (VDD), U1.47 (VDD), U1.6 (VBAT), U1.64 (VDD), U1.79 (VDD), U1.95 (VDD)
- new net +3.3VA: C12.1, C13.1, U1.45 (VDDA)
- new net A0: U1.18 (PF10), U2.5 (A0)
- new net A1: U1.15 (PF7), U2.4 (A1)
- new net A10: U2.29 (A10)
- new net A11: U2.28 (A11)
- new net A12: U2.27 (A12)
- new net A13: U1.70 (PD8), U2.26 (A13)
- new net A14: U1.71 (PD9), U2.25 (A14)
- new net A15: U1.103 (PG5), U1.72 (PD10), U2.24 (A15)
- new net A16: U1.73 (PD11), U2.23 (A16)
- new net A17: U1.74 (PD12), U2.22 (A17)
- new net A18: U1.75 (PD13), U2.21 (A18)
- new net A19: U1.2 (PE3), U2.20 (A19)
- new net A2: U1.26 (PF2), U2.3 (A2)
- new net A20: U1.3 (PE4), U2.31 (A20)
- new net A3: U1.10 (PF3), U2.2 (A3)
- new net A4: U1.11 (PF4), U2.1 (A4)
- new net A5: U1.14 (PF5), U2.48 (A5)
- new net A6: U1.49 (PF12), U2.47 (A6)
- new net A7: U1.50 (PF13), U2.46 (A7)
- new net A8: U1.51 (PF14), U2.45 (A8)
- new net A9: U1.52 (PF15), U2.30 (A9)
- new net GND: C1.2, C10.2, C11.2, C12.2, C13.2, C14.2, C15.2, C16.2, C17.2, C18.2, C19.2, C2.2, C3.2, C4.2, C5.2, C6.2, C7.2, C8.2, C9.2, J1.3 (Pin_3), R1.2, SW1.1 (A), U1.110 (VSS), U1.12 (VSS), U1.127 (VSS), U1.30 (VSS), U1.42 (VSSA), U1.46 (VSS), U1.63 (VSS), U1.78 (VSS), U1.94 (VSS), U2.13 (VSS), U2.37 (VSS), Y1.2 (G), Y1.4 (G)
- new net I/O0: U1.76 (PD14), U2.8 (I/O0)
- new net I/O1: U1.77 (PD15), U2.9 (I/O1)
- new net I/O10: U1.59 (PE13), U1.82 (PG0), U2.34 (I/O10)
- new net I/O11: U1.60 (PE14), U1.83 (PG1), U2.35 (I/O11)
- new net I/O12: U1.61 (PE15), U1.84 (PG2), U2.38 (I/O12)
- new net I/O13: U1.85 (PG3), U2.39 (I/O13)
- new net I/O14: U1.86 (PG4), U2.40 (I/O14)
- new net I/O15: U2.41 (I/O15)
- new net I/O2: U1.108 (PD0), U2.10 (I/O2)
- new net I/O3: U1.109 (PD1), U2.11 (I/O3)
- new net I/O4: U1.53 (PE7), U2.14 (I/O4)
- new net I/O5: U1.54 (PE8), U2.15 (I/O5)
- new net I/O6: U1.55 (PE9), U2.16 (I/O6)
- new net I/O7: U1.56 (PE10), U2.17 (I/O7)
- new net I/O8: U1.57 (PE11), U2.32 (I/O8)
- new net I/O9: U1.58 (PE12), U2.33 (I/O9)
- new net NRST: C16.1, R2.1, SW1.2 (B), U1.21 (PG10)
- new net OSC_IN: C1.1, U1.19 (PF0), Y1.1
- new net OSC_OUT: C2.1, U1.20 (PF1), Y1.3
- new net SWCLK: J1.1 (Pin_1), U1.93 (PA12)
- new net SWDIO: J1.2 (Pin_2), U1.96 (PA13)
- new net Trig: U1.65 (PB11)
- new net VCC: U2.12 (VDD), U2.36 (VDD)
- new net V_{REF}: C14.1, C15.1, U1.43 (VREF+), U1.44 (VREF_+)
- new net ~{CS}: U1.117 (PD7), U2.7 (CS#)
- new net ~{LB}: U1.125 (PE0), U2.42 (LB#)
- new net ~{OE}: U1.114 (PD4), U2.44 (OE#)
- new net ~{UB}: U1.126 (PE1), U2.43 (UB#)
- new net ~{WE}: U1.115 (PD5), U2.18 (WE#)
