File: hardware/MCU.kicad_sch (KiCad schematic)
At the start: 31 parts, among them J1 Conn_01x03_Pin, SW1 SW_MEC_5G, U1 STM32G473QETxZ, U2 IS61W204816BLL, U29 74LVC1G07, U30 GD25Q32JVSS, Y1 25MHz

Commit message: feat：电源原理图
Connections:
- net VCC is gone; now on net +3.3V: U2.12 (VDD), U2.36 (VDD)
Changed lines of the file:
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@@
 	)
 	(symbol
+		(lib_id "power:+3.3V")
+		(at 254 21.59 0)
+		(mirror y)
+		(unit 1)
+		(body_style 1)
+		(exclude_from_sim no)
+		(in_bom yes)
+		(on_board yes)
+		(in_pos_files yes)
+		(dnp no)
+		(property "Reference" "#PWR012"
+			(at 254 25.4 0)
+			(hide yes)
+			(show_name no)
+			(do_not_autoplace no)
+			(effects
+				(font
+					(size 1.27 1.27)
+				)
+			)
+		)
+		(property "Value" "+3.3V"
+			(at 254 16.51 0)
+			(show_name no)
+			(do_not_autoplace no)
+			(effects
+				(font
+					(size 1.27 1.27)
+				)
+			)
+		)
+		(property "Footprint" ""
+			(at 254 21.59 0)
+			(hide yes)
+			(show_name no)
+			(do_not_autoplace no)
+			(effects
+				(font
+					(size 1.27 1.27)
+				)
+			)
+		)
+		(property "Datasheet" ""
+			(at 254 21.59 0)
+			(hide yes)
+			(show_name no)
+			(do_not_autoplace no)
+			(effects
+				(font
+					(size 1.27 1.27)
+				)
+			)
+		)
+		(property "Description" "Power symbol creates a global label with name \"+3.3V\""
+			(at 254 21.59 0)
+			(hide yes)
+			(show_name no)
+			(do_not_autoplace no)
+			(effects
+				(font
+					(size 1.27 1.27)
+				)
+			)
+		)
+		(pin "1"
+		)
+		(instances
+			(project "E4"
+				(path "/7664cc8d-15c4-46a0-b3f4-8b4373008b19/7eca7ef4-dc42-4686-9d4a-c20d29fed480"
+					(reference "#PWR012")
+					(unit 1)
+				)
+			)
+		)
+	)
+	(symbol
 		(lib_id "Device:C")
 		(at 22.86 115.57 0)
@@
 					(unit 1)
 				)
-			)
-		)
-	)
-	(symbol
-		(lib_id "power:VCC")
-		(at 254 21.59 0)
-		(unit 1)
-		(body_style 1)
-		(exclude_from_sim no)
-		(in_bom yes)
-		(on_board yes)
-		(in_pos_files yes)
-		(dnp no)
-		(fields_autoplaced yes)
-		(property "Reference" "#PWR1"
-			(at 254 25.4 0)
-			(hide yes)
-			(show_name no)
-			(do_not_autoplace no)
-			(effects
-				(font
-					(size 1.27 1.27)
-				)
-			)
-		)
-		(property "Value" "VCC"
-			(at 254 16.51 0)
-			(show_name no)
-			(do_not_autoplace no)
-			(effects
-				(font
-					(size 1.27 1.27)
-				)
-			)
-		)
-		(property "Footprint" ""
-			(at 254 21.59 0)
-			(hide yes)
-			(show_name no)
-			(do_not_autoplace no)
-			(effects
-				(font
-					(size 1.27 1.27)
-				)
-			)
-		)
-		(property "Datasheet" ""
-			(at 254 21.59 0)
-			(hide yes)
-			(show_name no)
-			(do_not_autoplace no)
-			(effects
-				(font
-					(size 1.27 1.27)
-				)
-			)
-		)
-		(property "Description" "Power symbol creates a global label with name \"VCC\""
-			(at 254 21.59 0)
-			(hide yes)
-			(show_name no)
-			(do_not_autoplace no)
-			(effects
-				(font
-					(size 1.27 1.27)
-				)
-			)
-		)
-		(pin "1"
-		)
-		(instances
-			(project "E4"
-				(path "/7664cc8d-15c4-46a0-b3f4-8b4373008b19/7eca7ef4-dc42-4686-9d4a-c20d29fed480"
-					(reference "#PWR1")
-					(unit 1)
-				)

Commit message: feat：模拟前端布线，单片机/SRAM布线
Parts:
- C12, C13, C4: footprint Capacitor_SMD:C_0603_1608Metric -> Capacitor_SMD:C_0402_1005Metric
- J1: footprint (none) -> Connector_PinHeader_1.00mm:PinHeader_1x03_P1.00mm_Vertical
- U29: footprint (none) -> Package_TO_SOT_SMD:SOT-23-5
- Y1: footprint Crystal:Crystal_SMD_3225-4Pin_3.2x2.5mm -> Crystal:Crystal_SMD_2016-4Pin_2.0x1.6mm
Connections:
- net USART_RX is gone; now on net U.RXD: U1.91 (PA10)
- net USB_Check is gone; now on net USB.USB_Check: U1.89 (PA8)
- net USB_D+ is gone; now on net USB.USB_D+: U1.93 (PA12)
- net USB_D- is gone; now on net USB.USB_D-: U1.92 (PA11)
- no-connect marks 1 -> 38

Commit message: feat：电源部分
Parts:
- C1, C2: footprint Capacitor_SMD:C_0603_1608Metric -> Capacitor_SMD:C_0402_1005Metric
Connections:
- net Ctrl3: now reaches U1.7 (PC13)
- net Ctrl4: now reaches U1.8 (PC14)
- net Ctrl1: now reaches U1.4 (PE5)
- net Ctrl2: now reaches U1.5 (PE6)
- no-connect marks 38 -> 34
Changed lines of the file:
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@@
 	)
 	(no_connect
-		(at 187.96 146.05)
-	)
-	(no_connect
-		(at 224.79 124.46)
-	)
-	(no_connect
 		(at 134.62 40.64)
 	)
@@
 	)
 	(no_connect
-		(at 224.79 127)
-	)
-	(no_connect
 		(at 87.63 39.37)
 	)
@@
 	)
 	(no_connect
-		(at 187.96 143.51)
-	)
-	(no_connect
 		(at 218.44 45.72)
 	)
@@
 	(wire
 		(pts
+			(xy 190.5 143.51) (xy 187.96 143.51)
+		)
+		(stroke
+			(width 0)
+			(type default)
+		)
+	)
+	(wire
+		(pts
 			(xy 50.8 107.95) (xy 50.8 109.22)
 		)
@@
 	(wire
 		(pts
+			(xy 228.6 127) (xy 224.79 127)
+		)
+		(stroke
+			(width 0)
+			(type default)
+		)
+	)
+	(wire
+		(pts
 			(xy 236.22 38.1) (xy 243.84 38.1)
 		)
@@
 	(wire
 		(pts
+			(xy 190.5 146.05) (xy 187.96 146.05)
+		)
+		(stroke
+			(width 0)
+			(type default)
+		)
+	)
+	(wire
+		(pts
 			(xy 128.27 156.21) (xy 138.43 156.21)
 		)
@@
 	(wire
 		(pts
+			(xy 228.6 124.46) (xy 224.79 124.46)
+		)
+		(stroke
+			(width 0)
+			(type default)
+		)
+	)
+	(wire
+		(pts
 			(xy 224.79 149.86) (xy 232.41 149.86)
 		)
@@
 		)
 	)
+	(hierarchical_label "Ctrl4"
+		(shape input)
+		(at 190.5 146.05 0)
+		(effects
+			(font
+				(size 1.27 1.27)
+			)
+			(justify left)
+		)
+	)
 	(hierarchical_label "USART"
 		(shape input)
@@
 		)
 	)
+	(hierarchical_label "Ctrl2"
+		(shape input)
+		(at 228.6 127 0)
+		(effects
+			(font
+				(size 1.27 1.27)
+			)
+			(justify left)
+		)
+	)
 	(hierarchical_label "CH3-"
 		(shape input)
@@
 		)
 	)
+	(hierarchical_label "Ctrl3"
+		(shape input)
+		(at 190.5 143.51 0)
+		(effects
+			(font
+				(size 1.27 1.27)
+			)
+			(justify left)
+		)
+	)
 	(hierarchical_label "CH1+"
 		(shape input)
@@
 		)
 	)
+	(hierarchical_label "Ctrl1"
+		(shape input)
+		(at 228.6 124.46 0)
+		(effects
+			(font
+				(size 1.27 1.27)
+			)
+			(justify left)
+		)
+	)
 	(rule_area
 		(exclude_from_sim no)
@@
 			)
 		)
-		(property "Footprint" "Capacitor_SMD:C_0603_1608Metric"
+		(property "Footprint" "Capacitor_SMD:C_0402_1005Metric"
 			(at 21.8948 119.38 0)
 			(hide yes)
@@
 			)
 		)
-		(property "Footprint" "Capacitor_SMD:C_0603_1608Metric"
+		(property "Footprint" "Capacitor_SMD:C_0402_1005Metric"
 			(at 36.5252 119.38 0)
 			(hide yes)

Commit message: feat：总体连接
Connections:
- net V_{REF} renamed V_{REF_OUT}
Changed lines of the file:
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@@
 		)
 	)
-	(hierarchical_label "V_{REF}"
+	(hierarchical_label "V_{REF_OUT}"
 		(shape input)
 		(at 53.34 57.15 0)

Commit message: feat：整理设计文件
Parts:
- Y1: value 25MHz -> 24MHz
Changed lines of the file:
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@@
 			)
 		)
-		(property "Value" "25MHz"
+		(property "Value" "24MHz"
 			(at 29.21 101.6 0)
 			(show_name no)
