File: hardware/CH1,2.kicad_sch (KiCad schematic)
At the start: 104 parts, among them J2 RJ45, J3 RJ45, U10 ADG719, U11 INA828, U12 OPA2192, U13 OPA2192, U14 INA828, U15 SGM2059, U4 INA828, U5 OPA2192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

Commit message: feat：输入滤波原理图
Parts:
- removed C24, C25, C26, C35, C36, C37: 100pF, Capacitor_SMD:C_0603_1608Metric, symbol Device:C
- removed R15, R16, R29, R30: 49.9R, Resistor_SMD:R_0603_1608Metric, symbol Device:R

Commit message: feat：电平触发原理图
Parts:
- added C140, C141: 1uF, Capacitor_SMD:C_0603_1608Metric, symbol Device:C
Connections:
- net GND: now also C140.2, C141.2
- net V_{REF}: now also C140.1, C141.1

Commit message: feat：模拟前端布线，单片机/SRAM布线
Parts:
- added TP10: INA_O2, TestPoint:TestPoint_Pad_D1.0mm, symbol Connector:TestPoint
- added TP11: Filter_O1, TestPoint:TestPoint_Pad_D1.0mm, symbol Connector:TestPoint
- added TP12: Filter_O2, TestPoint:TestPoint_Pad_D1.0mm, symbol Connector:TestPoint
- added TP9: INA_O1, TestPoint:TestPoint_Pad_D1.0mm, symbol Connector:TestPoint
- U10, U9: footprint ProPrj_New Project_2026-05-28_15-29-15_2026-05-30:SOT-23-8_L3.0-W1.7-P0.65-LS2.8-TL -> Package_TO_SOT_SMD:SOT-23-8
- U11, U14, U4, U7: footprint Package_SO:Infineon_PG-DSO-8-43 -> Package_SO:SOIC-8_3.9x4.9mm_P1.27mm
Connections:
- net at C32.1, R25.2, R27.2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: now also TP12.1
- net at R7.2, U4.6 (OUT): now also TP9.1
- net at R21.2, U11.6 (OUT): now also TP10.1
- net at C23.1, R10.2, R11.2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: now also TP11.1

Commit message: feat：电源部分
Changed lines of the file:
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@@
+		)
+	)
+	(hierarchical_label "Ctrl1"
+		(shape input)
+		(at 62.23 50.8 180)
+		(effects
+			(font
+				(size 1.27 1.27)
+			)
+			(justify right)
+		)
+	)
+	(hierarchical_label "Ctrl2"
+		(shape input)
+		(at 63.5 96.52 180)
+		(effects
+			(font
+				(size 1.27 1.27)
+			)
+			(justify right)
 		)
 	)

Commit message: feat：总体连接
Connections:
- net +2.5VA is gone; now on net V_{REF}: C136.2, C137.2, R18.1, R4.1
Changed lines of the file:
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@@
 	(global_label "V_{REF}"
 		(shape input)
+		(at 52.07 17.78 180)
+		(fields_autoplaced yes)
+		(effects
+			(font
+				(size 1.27 1.27)
+			)
+			(justify right)
+		)
+		(property "Intersheetrefs" "${INTERSHEET_REFS}"
+			(at 45.1393 17.78 0)
+			(hide yes)
+			(show_name no)
+			(do_not_autoplace no)
+			(effects
+				(font
+					(size 1.27 1.27)
+				)
+				(justify right)
+			)
+		)
+	)
+	(global_label "V_{REF}"
+		(shape input)
 		(at 250.19 50.8 180)
 		(fields_autoplaced yes)
@@
 	(global_label "V_{REF}"
 		(shape input)
+		(at 53.34 63.5 180)
+		(fields_autoplaced yes)
+		(effects
+			(font
+				(size 1.27 1.27)
+			)
+			(justify right)
+		)
+		(property "Intersheetrefs" "${INTERSHEET_REFS}"
+			(at 46.4093 63.5 0)
+			(hide yes)
+			(show_name no)
+			(do_not_autoplace no)
+			(effects
+				(font
+					(size 1.27 1.27)
+				)
+				(justify right)
+			)
+		)
+	)
+	(global_label "V_{REF}"
+		(shape input)
 		(at 217.17 101.6 180)
 		(fields_autoplaced yes)
@@
 	)
 	(symbol
-		(lib_id "power:+4V")
-		(at 52.07 17.78 90)
-		(unit 1)
-		(body_style 1)
-		(exclude_from_sim no)
-		(in_bom yes)
-		(on_board yes)
-		(in_pos_files yes)
-		(dnp no)
-		(fields_autoplaced yes)
-		(property "Reference" "#PWR122"
-			(at 55.88 17.78 0)
-			(hide yes)
-			(show_name no)
-			(do_not_autoplace no)
-			(effects
-				(font
-					(size 1.27 1.27)
-				)
-			)
-		)
-		(property "Value" "+2.5VA"
-			(at 48.26 17.7799 90)
-			(show_name no)
-			(do_not_autoplace no)
-			(effects
-				(font
-					(size 1.27 1.27)
-				)
-				(justify left)
-			)
-		)
-		(property "Footprint" ""
-			(at 52.07 17.78 0)
-			(hide yes)
-			(show_name no)
-			(do_not_autoplace no)
-			(effects
-				(font
-					(size 1.27 1.27)
-				)
-			)
-		)
-		(property "Datasheet" ""
-			(at 52.07 17.78 0)
-			(hide yes)
-			(show_name no)
-			(do_not_autoplace no)
-			(effects
-				(font
-					(size 1.27 1.27)
-				)
-			)
-		)
-		(property "Description" "Power symbol creates a global label with name \"+4V\""
-			(at 52.07 17.78 0)
-			(hide yes)
-			(show_name no)
-			(do_not_autoplace no)
-			(effects
-				(font
-					(size 1.27 1.27)
-				)
-			)
-		)
-		(pin "1"
-		)
-		(instances
-			(project "E4"
-				(path "/7664cc8d-15c4-46a0-b3f4-8b4373008b19/19d13e66-38d6-49c3-ac36-dcbde1979dd4"
-					(reference "#PWR122")
-					(unit 1)
-				)
-			)
-		)
-	)
-	(symbol
 		(lib_id "Device:C")
 		(at 168.91 162.56 0)
@@
 					(unit 1)
 				)
-			)
-		)
-	)
-	(symbol
-		(lib_id "power:+4V")
-		(at 53.34 63.5 90)
-		(unit 1)
-		(body_style 1)
-		(exclude_from_sim no)
-		(in_bom yes)
-		(on_board yes)
-		(in_pos_files yes)
-		(dnp no)
-		(fields_autoplaced yes)
-		(property "Reference" "#PWR25"
-			(at 57.15 63.5 0)
-			(hide yes)
-			(show_name no)
-			(do_not_autoplace no)
-			(effects
-				(font
-					(size 1.27 1.27)
-				)
-			)
-		)
-		(property "Value" "+2.5VA"
-			(at 49.53 63.4999 90)
-			(show_name no)
-			(do_not_autoplace no)
-			(effects
-				(font
-					(size 1.27 1.27)
-				)
-				(justify left)
-			)
-		)
-		(property "Footprint" ""
-			(at 53.34 63.5 0)
-			(hide yes)
-			(show_name no)
-			(do_not_autoplace no)
-			(effects
-				(font
-					(size 1.27 1.27)
-				)
-			)
-		)
-		(property "Datasheet" ""
-			(at 53.34 63.5 0)
-			(hide yes)
-			(show_name no)
-			(do_not_autoplace no)
-			(effects
-				(font
-					(size 1.27 1.27)
-				)
-			)
-		)
-		(property "Description" "Power symbol creates a global label with name \"+4V\""
-			(at 53.34 63.5 0)
-			(hide yes)
-			(show_name no)
-			(do_not_autoplace no)
-			(effects
-				(font
-					(size 1.27 1.27)
-				)
-			)
-		)
-		(pin "1"
-		)
-		(instances
-			(project "E4"
-				(path "/7664cc8d-15c4-46a0-b3f4-8b4373008b19/19d13e66-38d6-49c3-ac36-dcbde1979dd4"
-					(reference "#PWR25")
-					(unit 1)
-				)
