File: hardware/E4.kicad_pcb (KiCad board)
At the start: 4 copper layers, 170 x 115 mm, 305 parts, among them J1 Conn_01x03_Pin, J2 RJ45, J3 RJ45, J4 RJ45, J5 RJ45, J6 USB_A_Stacked, J7 Barrel_Jack_Switch, SW1 SW_MEC_5G, SW2 PS-22F02, U1 STM32G473QETxZ, U10 ADG719, U11 INA828, U12 OPA2192, U13 OPA2192, U14 INA828, U15 SGM2059, U16 INA828, U17 SGM2059, U18 ADG719, U19 ADG719, U2 IS61W204816BLL, U20 INA828, U21 INA828, U22 INA828, U23 SGM2059, U24 OPA2192, U25 OPA2192, U26 OPA2192, U27 OPA2192, U28 OPA197xDBV, U29 74LVC1G07, U3 ADG704BRMZ, U30 GD25Q32JVSS, U31 SGM3204, U32 TPS7A4701xRGW, U33 TPS7A3301RGW, U34 AMS1117-3.3, U35 SGM2059, U4 INA828, U5 OPA2192, U6 OPA2192, U7 INA828, U8 SGM2059, U9 ADG719, Y1 25MHz

Commit message: feat：电源部分
Parts:
- added C163: 10uF, Capacitor_SMD:C_0603_1608Metric, F.Cu at (157.0, 126.2)
- added C165: 100nF, Capacitor_SMD:C_0603_1608Metric, F.Cu at (158.5, 126.2)
- added D3: SMBJ5A, Diode_SMD:D_SMF, F.Cu at (132.5, 104.1)
- C145, C146, C166, C167, D2, R1, R65, R66, U29: moved to B.Cu
- moved C151 189.1 mm to (122.9, 33.3)
- moved C169 187.0 mm to (122.9, 31.4), turned to 180 degrees
- moved TP3 185.3 mm to (119.3, 33.3), turned to 90 degrees
- moved U32 183.0 mm to (124.4, 37.7)
- moved R1 179.5 mm to (103.2, 60.0), turned to 90 degrees
- moved C166 174.9 mm to (129.4, 37.0), turned to 180 degrees
- moved C152 174.5 mm to (128.2, 34.5), turned to 90 degrees
- moved J7 169.9 mm to (135.6, 101.7)
- moved SW2 169.7 mm to (141.0, 87.1)
- moved J6 169.6 mm to (139.3, 69.2)
- moved D2 165.9 mm to (132.6, 65.7), turned to -90 degrees
- moved R63 165.2 mm to (132.8, 69.5)
- moved R64 164.8 mm to (132.8, 68.0)
- moved U29 162.8 mm to (128.0, 67.6)
- moved D1 162.6 mm to (132.6, 65.7), turned to -90 degrees
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Connections:
- D1 pad 2: /USB.USB_D- -> /USB.USB_D+
- D1 pad 3: /USB.USB_D+ -> /USB.USB_D-
- D2 pad 1: unconnected-(D2-GND-Pad1) -> GND
- D2 pad 2: /U.TXD -> /U.RXD
- D2 pad 3: /U.RXD -> /U.TXD
- D2 pad 4: unconnected-(D2-VCC-Pad4) -> VBUS
- J6 pad 2: /USB.USB_D- -> /U.TXD
- J6 pad 3: /USB.USB_D+ -> /U.RXD
- J6 pad 6: /U.TXD -> /USB.USB_D-
- J6 pad 7: /U.RXD -> /USB.USB_D+
- U1 pad 4: unconnected-(U1F-PE5-Pad4) -> /CH1,2/Ctrl1
- U1 pad 5: unconnected-(U1F-PE6-Pad5) -> /CH1,2/Ctrl2
- U1 pad 7: unconnected-(U1D-PC13-Pad7) -> /CH3,4/Ctrl3
- U1 pad 8: unconnected-(U1D-PC14-Pad8) -> /CH3,4/Ctrl4
Routing:
- net /MCU/A3: track 0.05 -> 61.5 mm, vias 0 -> 2
- net /MCU/A4: track 0.00 -> 51.6 mm, vias 0 -> 2
- net /MCU/TRIG: track 0.00 -> 51.5 mm, vias 0 -> 2
- net /U.RXD: track 0.00 -> 28.9 mm, vias 0 -> 1
- net /MCU/CTrig1: track 0.00 -> 28.2 mm
- net /MCU/CTrig0: track 0.00 -> 24.9 mm
- net /USB.USB_D-: track 0.00 -> 22.5 mm
- net /USB.USB_D+: track 0.00 -> 22.5 mm
- net /MCU/NRST: track 1.21 -> 22.8 mm, vias 1 -> 3
- net /MCU/USART_TX: track 0.00 -> 12.0 mm, vias 0 -> 1
- net +3.3V: track 23.8 -> 35.7 mm, vias 9 -> 16
- net /U.TXD: track 0.00 -> 11.8 mm
- net Net-(U31-CFLY-): track 0.00 -> 5.79 mm
- net VCC: track 0.00 -> 5.26 mm, vias 0 -> 5
- net GND: track 0.02 -> 5.23 mm, vias 1 -> 9
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- added copper zone on F.Cu, net +3.3VA
- added copper zone on F.Cu, net +4VA
- added copper zone on F.Cu, net -4VA
- added copper zone on F.Cu, net -5VA
- added copper zone on B.Cu, net GND
- added copper zone on F.Cu, net GND
- added copper zone on B.Cu, net VBUS
- added copper zone on F.Cu, net VBUS
- added copper zone on F.Cu, net VCC
- added copper zone on F.Cu, net V_{IN}
Other:
- board size 170 x 115 mm -> 130 x 115 mm

Commit message: feat：总体连接
Parts:
- moved C14 89.8 mm to (81.6, 81.2), turned to -90 degrees
- moved C15 89.8 mm to (83.1, 81.2), turned to -90 degrees
- moved C165 89.6 mm to (79.1, 84.6)
- moved U28 89.6 mm to (78.7, 81.4)
- moved C163 89.6 mm to (77.6, 84.6)
- moved TP2 89.6 mm to (75.2, 80.4)
- moved TP21 1.37 mm to (74.0, 128.2)
- moved TP22 1.26 mm to (77.2, 128.3)
- moved TP19 0.86 mm to (74.1, 101.1)
- moved TP20 0.80 mm to (77.2, 101.1)
- moved TP18 0.57 mm to (77.1, 74.6)
- moved TP17 0.53 mm to (74.2, 74.5)
- moved TP15 0.41 mm to (74.1, 48.0)
- moved TP16 0.41 mm to (77.1, 48.0)
- moved C56 0.11 mm to (49.1, 31.4)
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Connections:
- C136 pad 2: +2.5VA -> V_{REF}
- C137 pad 2: +2.5VA -> V_{REF}
- C138 pad 2: +2.5VA -> V_{REF}
- C139 pad 2: +2.5VA -> V_{REF}
- C14 pad 1: V_{REF} -> /MCU/V_{REF_OUT}
- C15 pad 1: V_{REF} -> /MCU/V_{REF_OUT}
- R18 pad 1: +2.5VA -> V_{REF}
- R34 pad 1: +2.5VA -> V_{REF}
- R35 pad 1: +2.5VA -> V_{REF}
- R4 pad 1: +2.5VA -> V_{REF}
- R63 pad 2: /USB.VBUS_Check -> /USB.USB_Check
- R64 pad 2: /USB.VBUS_Check -> /USB.USB_Check
- U1 pad 43: V_{REF} -> /MCU/V_{REF_OUT}
- U1 pad 44: V_{REF} -> /MCU/V_{REF_OUT}
- U28 pad 3: V_{REF} -> /MCU/V_{REF_OUT}
Routing:
- net V_{REF}: track 36.7 -> 291.3 mm, vias 12 -> 17
- net /CH3,4/Ctrl4: track 1.77 -> 114.5 mm, vias 1 -> 2
- net /CH3,4/D4Q+: track 3.31 -> 99.1 mm, vias 1 -> 3
- net /CH3,4/Ctrl3: track 1.77 -> 92.0 mm, vias 1 -> 2
- net /CH3,4/D3Q+: track 1.27 -> 72.6 mm, vias 0 -> 3
- net /CH3,4/D4Q-: track 4.16 -> 75.2 mm, vias 1 -> 2
- net /CH1,2/Ctrl2: track 1.77 -> 71.7 mm, vias 1 -> 2
- net /CH1,2/Ctrl1: track 1.77 -> 68.4 mm, vias 1 -> 2
- net /CH1,2/D1Q+: track 5.15 -> 67.9 mm, vias 1 -> 2
- net /CH1,2/D1Q-: track 6.35 -> 59.8 mm, vias 1 -> 2
- net /CH3,4/D3Q-: track 2.10 -> 54.7 mm, vias 0 -> 2
- net +4VA: track 69.3 -> 111.4 mm, vias 25 -> 30
- net +3.3VA: track 3.85 -> 38.3 mm
- net /CH1,2/D2Q+: track 8.53 -> 41.7 mm, vias 1 -> 3
- net /CH1,2/D2Q-: track 9.24 -> 36.8 mm, vias 1 -> 2
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- added copper zone on In2.Cu, net +3.3V
- added copper zone on In2.Cu, net +4VA
- added copper zone on In2.Cu, net -4VA
- added copper zone on In2.Cu, net /CH1,2/EX1+
- added copper zone on In2.Cu, net /CH1,2/EX2+
- added copper zone on In2.Cu, net /CH3,4/EX3+
- added copper zone on In2.Cu, net /CH3,4/EX4+
- added copper zone on F.Cu, net /MCU/V_{REF_OUT}
- added copper zone on In2.Cu, net VCC
