File: hardware/E4.kicad_pcb (KiCad board)
At the start: 4 copper layers, 130 x 115 mm, 308 parts, among them J1 Conn_01x03_Pin, J2 RJ45, J3 RJ45, J4 RJ45, J5 RJ45, J6 USB_A_Stacked, J7 Barrel_Jack_Switch, SW1 SW_MEC_5G, SW2 PS-22F02, U1 STM32G473QETxZ, U10 ADG719, U11 INA828, U12 OPA2192, U13 OPA2192, U14 INA828, U15 SGM2059, U16 INA828, U17 SGM2059, U18 ADG719, U19 ADG719, U2 IS61W204816BLL, U20 INA828, U21 INA828, U22 INA828, U23 SGM2059, U24 OPA2192, U25 OPA2192, U26 OPA2192, U27 OPA2192, U28 OPA197xDBV, U29 74LVC1G07, U3 ADG704BRMZ, U30 GD25Q32JVSS, U31 SGM3204, U32 TPS7A4701xRGW, U33 TPS7A3301RGW, U34 AMS1117-3.3, U35 SGM2059, U4 INA828, U5 OPA2192, U6 OPA2192, U7 INA828, U8 SGM2059, U9 ADG719, Y1 25MHz

Commit message: feat：整理设计文件
Parts:
- Y1: value 25MHz -> 24MHz
Changed lines of the file:
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@@
 			)
 		)
-		(property "Value" "25MHz"
+		(property "Value" "24MHz"
 			(at 0 2 270)
 			(layer "F.Fab")
@@
 	)
 	(segment
+		(start 131.9286 69.5452)
+		(end 131.9286 68.0466)
+		(width 0.254)
+		(layer "F.Cu")
+		(net "/USB.USB_Check")
+	)
+	(segment
+		(start 115.2345 67.070751)
+		(end 122.163351 67.070751)
+		(width 0.254)
+		(layer "F.Cu")
+		(net "/USB.USB_Check")
+	)
+	(segment
+		(start 122.163351 67.070751)
+		(end 124.6378 69.5452)
+		(width 0.254)
+		(layer "F.Cu")
+		(net "/USB.USB_Check")
+	)
+	(segment
+		(start 124.6378 69.5452)
+		(end 131.9286 69.5452)
+		(width 0.254)
+		(layer "F.Cu")
+		(net "/USB.USB_Check")
+	)
+	(segment
 		(start 42.85305 28.51835)
 		(end 38.42245 28.51835)
@@
 	)
 	(segment
+		(start 83.0495 80.4465)
+		(end 83.0696 80.4666)
+		(width 0.4064)
+		(layer "F.Cu")
+		(net "/MCU/V_{REF_OUT}")
+	)
+	(segment
+		(start 79.874684 80.4465)
+		(end 83.0495 80.4465)
+		(width 0.4064)
+		(layer "F.Cu")
+		(net "/MCU/V_{REF_OUT}")
+	)
+	(segment
+		(start 84.937 80.4666)
+		(end 84.963 80.4926)
+		(width 0.4064)
+		(layer "F.Cu")
+		(net "/MCU/V_{REF_OUT}")
+	)
+	(segment
+		(start 83.0696 80.4666)
+		(end 84.937 80.4666)
+		(width 0.4064)
+		(layer "F.Cu")
+		(net "/MCU/V_{REF_OUT}")
+	)
+	(via
+		(at 84.963 80.4926)
+		(size 0.6096)
+		(drill 0.3048)
+		(layers "F.Cu" "B.Cu")
+		(net "/MCU/V_{REF_OUT}")
+	)
+	(via
+		(at 103.3526 76.3524)
+		(size 0.6096)
+		(drill 0.3048)
+		(layers "F.Cu" "B.Cu")
+		(free yes)
+		(net "/MCU/V_{REF_OUT}")
+	)
+	(segment
+		(start 95.594449 80.122751)
+		(end 85.332849 80.122751)
+		(width 0.4064)
+		(layer "In2.Cu")
+		(net "/MCU/V_{REF_OUT}")
+	)
+	(segment
+		(start 85.332849 80.122751)
+		(end 84.963 80.4926)
+		(width 0.4064)
+		(layer "In2.Cu")
+		(net "/MCU/V_{REF_OUT}")
+	)
+	(segment
+		(start 103.3526 77.2922)
+		(end 101.7016 78.9432)
+		(width 0.4064)
+		(layer "In2.Cu")
+		(net "/MCU/V_{REF_OUT}")
+	)
+	(segment
+		(start 101.7016 78.9432)
+		(end 96.774 78.9432)
+		(width 0.4064)
+		(layer "In2.Cu")
+		(net "/MCU/V_{REF_OUT}")
+	)
+	(segment
+		(start 103.3526 76.3524)
+		(end 103.3526 77.2922)
+		(width 0.4064)
+		(layer "In2.Cu")
+		(net "/MCU/V_{REF_OUT}")
+	)
+	(segment
+		(start 96.774 78.9432)
+		(end 95.594449 80.122751)
+		(width 0.4064)
+		(layer "In2.Cu")
+		(net "/MCU/V_{REF_OUT}")
+	)
+	(segment
 		(start 106.20412 87.644631)
 		(end 105.921 87.644631)
@@
 	)
 	(segment
-		(start 131.9286 69.5452)
-		(end 131.9286 68.0466)
-		(width 0.254)
-		(layer "F.Cu")
-		(net "/USB.USB_Check")
-	)
-	(segment
-		(start 115.2345 67.070751)
-		(end 122.163351 67.070751)
-		(width 0.254)
-		(layer "F.Cu")
-		(net "/USB.USB_Check")
-	)
-	(segment
-		(start 122.163351 67.070751)
-		(end 124.6378 69.5452)
-		(width 0.254)
-		(layer "F.Cu")
-		(net "/USB.USB_Check")
-	)
-	(segment
-		(start 124.6378 69.5452)
-		(end 131.9286 69.5452)
-		(width 0.254)
-		(layer "F.Cu")
-		(net "/USB.USB_Check")
-	)
-	(segment
 		(start 123.058751 66.670751)
 		(end 115.2345 66.670751)
@@
 		(net "Net-(U33-NR{slash}SS)")
 	)
-	(segment
-		(start 83.0495 80.4465)
-		(end 83.0696 80.4666)
-		(width 0.4064)
-		(layer "F.Cu")
-		(net "/MCU/V_{REF_OUT}")
-	)
-	(segment
-		(start 79.874684 80.4465)
-		(end 83.0495 80.4465)
-		(width 0.4064)
-		(layer "F.Cu")
-		(net "/MCU/V_{REF_OUT}")
-	)
-	(segment
-		(start 84.937 80.4666)
-		(end 84.963 80.4926)
-		(width 0.4064)
-		(layer "F.Cu")
-		(net "/MCU/V_{REF_OUT}")
-	)
-	(segment
-		(start 83.0696 80.4666)
-		(end 84.937 80.4666)
-		(width 0.4064)
-		(layer "F.Cu")
-		(net "/MCU/V_{REF_OUT}")
-	)
-	(via
-		(at 84.963 80.4926)
-		(size 0.6096)
-		(drill 0.3048)
-		(layers "F.Cu" "B.Cu")
-		(net "/MCU/V_{REF_OUT}")
-	)
-	(via
-		(at 103.3526 76.3524)
-		(size 0.6096)
-		(drill 0.3048)
-		(layers "F.Cu" "B.Cu")
-		(free yes)
-		(net "/MCU/V_{REF_OUT}")
-	)
-	(segment
-		(start 95.594449 80.122751)
-		(end 85.332849 80.122751)
-		(width 0.4064)
-		(layer "In2.Cu")
-		(net "/MCU/V_{REF_OUT}")
-	)
-	(segment
-		(start 85.332849 80.122751)
-		(end 84.963 80.4926)
-		(width 0.4064)
-		(layer "In2.Cu")
-		(net "/MCU/V_{REF_OUT}")
-	)
-	(segment
-		(start 103.3526 77.2922)
-		(end 101.7016 78.9432)
-		(width 0.4064)
-		(layer "In2.Cu")
-		(net "/MCU/V_{REF_OUT}")
-	)
-	(segment
-		(start 101.7016 78.9432)
-		(end 96.774 78.9432)
-		(width 0.4064)
-		(layer "In2.Cu")
-		(net "/MCU/V_{REF_OUT}")
-	)
-	(segment
-		(start 103.3526 76.3524)
-		(end 103.3526 77.2922)
-		(width 0.4064)
-		(layer "In2.Cu")
-		(net "/MCU/V_{REF_OUT}")
-	)
-	(segment
-		(start 96.774 78.9432)
-		(end 95.594449 80.122751)
-		(width 0.4064)
-		(layer "In2.Cu")
-		(net "/MCU/V_{REF_OUT}")
-	)
 	(zone
