File: hardware/power.kicad_sch (KiCad schematic)
At the start: 32 parts, among them U28 OPA197xDBV, U32 TPS7A4701xRGW, U33 TPS7A3301RGW, U34 AMS1117-3.3, U35 SGM2059

Commit message: feat：模拟前端布线，单片机/SRAM布线
Parts:
- added TP1: -5VA, TestPoint:TestPoint_Pad_D1.0mm, symbol Connector:TestPoint
- added TP2: V_{REF}, TestPoint:TestPoint_Pad_D1.0mm, symbol Connector:TestPoint
- added TP3: +4VA, TestPoint:TestPoint_Pad_D1.0mm, symbol Connector:TestPoint
- added TP4: +3.3V, TestPoint:TestPoint_Pad_D1.0mm, symbol Connector:TestPoint
- added TP5: -4VA, TestPoint:TestPoint_Pad_D1.0mm, symbol Connector:TestPoint
- added TP6: +3.3VA, TestPoint:TestPoint_Pad_D1.0mm, symbol Connector:TestPoint
- U31: value (none) -> SGM3204
Connections:
- net +3.3V: now also TP4.1
- net +3.3VA: now also TP6.1
- net +4VA: now also TP3.1
- net -4VA: now also TP5.1
- net -5VA: now also TP1.1
- net GND: now also U32.9 (0.8V); no longer U32.12 (0.1V)
- net V_{REF}: now also TP2.1
- no-connect marks 0 -> 5

Commit message: feat：电源部分
Parts:
- added C163: 10uF, Capacitor_SMD:C_0603_1608Metric, symbol Device:C
- added C165: 100nF, Capacitor_SMD:C_0603_1608Metric, symbol Device:C
Connections:
- net +4VA: now also C163.1, C165.2
- net GND: now also C163.2, C165.1

Commit message: feat：总体连接
Connections:
- net V_{REF}: no longer C14.1, C15.1, U28.3 (+)
- new net V_{REF_OUT}: C14.1, C15.1, U28.3 (+)
Changed lines of the file:
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@@
 		)
 	)
-	(hierarchical_label "V_{REF}"
+	(hierarchical_label "V_{REF_OUT}"
 		(shape input)
 		(at 135.89 38.1 180)
