File: hardware/.history/CH1,2.kicad_sch (KiCad schematic)
At the start: 41 parts, among them J2 RJ45, U3 ADG719, U4 INA828, U5 OPA2192, U6 OPA2192

Commit message: feat：差分转单端原理图
Parts:
- added U7: INA828, Package_SO:Infineon_PG-DSO-8-43, symbol Amplifier_Instrumentation:INA828IDR
Connections:
- net +4VA: now also U7.7 (+VS)
- net -4VA: now also U7.4 (-VS)
- net GND: now also U7.5 (REF)
- net RS1+: now also U7.3 (+IN)
- net RS1-: now also U7.2 (-IN)
- no-connect marks 0 -> 2

Commit message: feat：远程感测原理图；多路通道
Parts:
- removed C38, C39: 10uF, Capacitor_SMD:C_0603_1608Metric, symbol Device:C
- removed C40, C41, C42, C43: 100nF, Capacitor_SMD:C_0603_1608Metric, symbol Device:C
- removed U3: ADG719, Package_TO_SOT_SMD:SOT-23-6, symbol Analog_Switch:ADG719BRTZ-REEL7
- added C136, C137, C27: 1uF, Capacitor_SMD:C_0603_1608Metric, symbol Device:C
- added C44, C47, C58, C59, C60, C61, C62, C63, C64, C65, C66, C67, C68, C69, C70, C72, C74, C76, C81, C83: 10uF, Capacitor_SMD:C_0603_1608Metric, symbol Device:C
- added C45, C46, C48, C49, C50, C51, C52, C53, C54, C55, C56, C57, C71, C73, C75, C77, C78, C79, C80, C82: 100nF, Capacitor_SMD:C_0603_1608Metric, symbol Device:C
- added J3: RJ45, Connector_RJ:RJ45_Amphenol_54602-x08_Horizontal, symbol Connector:RJ45
- added R13, R31: 26.7kR, Resistor_SMD:R_0603_1608Metric, symbol Device:R
- added R17, R32: 12.4kR, Resistor_SMD:R_0603_1608Metric, symbol Device:R
- added R18, R19, R26, R28: 1kR, Resistor_SMD:R_0603_1608Metric, symbol Device:R
- added R20: 120R, Resistor_SMD:R_0603_1608Metric, symbol Device:R
- added R21: 6.19kR, Resistor_SMD:R_0603_1608Metric, symbol Device:R
- added R22: 8.45kR, Resistor_SMD:R_0603_1608Metric, symbol Device:R
- added R23: 2.15kR, Resistor_SMD:R_0603_1608Metric, symbol Device:R
- added R24: 3.92kR, Resistor_SMD:R_0603_1608Metric, symbol Device:R
- added R25: 7kR, Resistor_SMD:R_0603_1608Metric, symbol Device:R
- added R27: 8kR, Resistor_SMD:R_0603_1608Metric, symbol Device:R
- added R29, R30: 49.9R, Resistor_SMD:R_0603_1608Metric, symbol Device:R
- added U10, U9: ADG719, ProPrj_New Project_2026-05-28_15-29-15_2026-05-30:SOT-23-8_L3.0-W1.7-P0.65-LS2.8-TL, symbol Analog_Switch:ADG619BRTZ-REEL7
- added U11, U14: INA828, Package_SO:Infineon_PG-DSO-8-43, symbol Amplifier_Instrumentation:INA828IDR
- added U12, U13: OPA2192, Package_SO:SOIC-8_3.9x4.9mm_P1.27mm, symbol Amplifier_Operational:OPA2192IDR
- added U15, U8: SGM2059, Package_TO_SOT_SMD:SOT-23-5, symbol Regulator_Linear:SGM2059-ADJXN5G/TR
- C28, C33: value 10uF -> 1uF
- C29, C31, C35: value 100nF -> 100pF
- C30: value 10uF -> 120pF
- C32: value 10uF -> 750pF
- C34: value 100nF -> 1uF
- C36, C37: value 10uF -> 100pF
- R12: value 8kR -> 1kR
- R14: value 7kR -> 1kR
- R3, R4: value 120R -> 1kR
Connections:
- net CH+ is gone; now on net CH1+: U4.3 (+IN)
- net EX1- is gone; now on net GND: J2.2, J2.7
- net +2.5VA: now also C136.2, C137.2, R18.1
- net +4VA: now also C46.2, C47.2, C48.2, C49.2, C50.2, C51.2, C56.2, C58.1, C59.1, C61.1, C62.1, C66.1, C68.1, C70.1, C72.1, C73.2, C74.1, C75.1, C76.1, C77.1, C78.1, C79.1, C82.2, C83.2, U10.4 (VDD), U11.7 (+VS), U12.4 (VSS), U13.4 (VSS), U14.7 (+VS), U15.1 (IN), U15.3 (EN), U8.1 (IN), U8.3 (EN), U9.4 (VDD); no longer C28.1, C29.1, C30.1, C31.1, C32.1, C33.1, C34.1, C35.1
- net -4VA: now also C52.1, C53.1, C54.1, C55.1, C57.1, C60.2, C63.2, C64.2, C65.2, C67.2, C69.2, C71.1, U10.7 (VSS), U11.4 (-VS), U14.4 (-VS), U9.7 (VSS); no longer C36.1, C37.1, U5.8 (VDD), U6.8 (VDD)
- net CH1-: now also U9.2 (S1)
- net Ctrl1: now also U9.6 (IN)
- net EX1+: now also C44.2, C45.2, U8.5 (OUT)
- net GND: now also C35.1, U5.8 (VDD), U6.8 (VDD), C136.1, C137.1, C27.2, C44.1, C45.1, C46.1, C47.1, C48.1, C49.1, C50.1, C51.1, C52.2, C53.2, C54.2, C55.2, C56.1, C57.2, C58.2, C59.2, C60.1, C61.2, C62.2, C63.1, C64.1, C65.1, C66.2, C67.1, C68.2, C69.1, C70.2, C71.2, C72.2, C73.1, C74.2, C75.2, C76.2, C77.2, C78.2, C79.2, C80.1, C81.1, C82.1, C83.1, J3.2, J3.7, R17.1, R19.2, R32.1, U10.3 (GND), U12.8 (VDD), U13.8 (VDD), U14.5 (REF), U15.2 (GND), U8.2 (GND), U9.3 (GND); no longer C30.2, C32.2, C35.2, C36.2
- net V_{REF}: now also C28.1, C33.1, C34.1, C27.1, R26.1, U11.5 (REF), U13.5 (VINB+)
- net at R3.1, R4.2: now also U9.8 (S2)
- net at U4.2 (-IN): now also U9.1 (D)
- net OUT1+: now reaches C24.1, C25.2, R15.1
- net OUT1-: now reaches C24.2, C26.1, R16.1
- net at U7.6 (OUT): now also R13.1
- new net: U10.1 (D), U11.2 (-IN)
- new net: R18.2, R19.1, U10.8 (S2)
- new net: C29.1, R22.1, U12.3 (VINA+)
- new net: C31.1, R24.1, U12.5 (VINB+)
- new net: R27.1, R28.2, U13.6 (VINB-)
- new net: R25.1, R26.2, U13.3 (VINA+)
- new net: R13.2, R17.2, U8.4 (FB)
- new net: C32.1, R25.2, R27.2, U12.6 (VINB-), U12.7 (VOUTB)
- new net: C30.1, R23.2, U12.1 (VOUTA), U12.2 (VINA-)
- new net: C30.2, R21.1, R22.2
- new net: R31.1, U14.6 (OUT)
- new net: R31.2, R32.2, U15.4 (FB)
- new net: C32.2, R23.1, R24.2
- new net: R20.2, U11.1 (RG)
- new net: R21.2, U11.6 (OUT)
- new net: R20.1, U11.8 (RG)
- new net CH2+: J3.4, U11.3 (+IN)
- new net CH2-: J3.5, U10.2 (S1)
- new net Ctrl2: U10.6 (IN)
- new net D2Q+: R29.2, U13.1 (VOUTA), U13.2 (VINA-)
- new net D2Q-: R28.1, R30.2, U13.7 (VOUTB)
- new net EX2+: C80.2, C81.2, J3.1, J3.8, U15.5 (OUT)
- new net OUT2+: C35.2, C36.1, R29.1
- new net OUT2-: C36.2, C37.1, R30.1
- new net RS2+: J3.3, U14.3 (+IN)
- new net RS2-: J3.6, U14.2 (-IN)
- no-connect marks 2 -> 6
Other:
- moved on the sheet: C20, C21, C22, C23, C24, C25, C26, J2, R10, R11, R12, R14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
