File: hardware/.history/E4.kicad_sch (KiCad schematic)
At the start: 0 parts

Commit message: feat：远程感测原理图；多路通道
Other:
- added sheet CH3,4 (CH3,4.kicad_sch)
Changed lines of the file:
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@@
 	(paper "A4")
 	(sheet
-		(at 72.39 22.86)
-		(size 19.05 16.51)
+		(at 43.18 33.02)
+		(size 19.05 15.24)
 		(exclude_from_sim no)
 		(in_bom yes)
@@
 		)
 		(property "Sheetname" "CH1,2"
-			(at 72.39 22.1484 0)
+			(at 43.18 32.3084 0)
 			(show_name no)
 			(do_not_autoplace no)
@@
 		)
 		(property "Sheetfile" "CH1,2.kicad_sch"
-			(at 72.39 39.9546 0)
+			(at 43.18 48.8446 0)
 			(show_name no)
 			(do_not_autoplace no)
@@
 	)
 	(sheet
-		(at 35.56 29.21)
-		(size 26.67 21.59)
+		(at 69.85 35.56)
+		(size 27.94 33.02)
 		(exclude_from_sim no)
 		(in_bom yes)
@@
 		)
 		(property "Sheetname" "MCU"
-			(at 35.56 28.4984 0)
+			(at 69.85 34.8484 0)
 			(show_name no)
 			(do_not_autoplace no)
@@
 		)
 		(property "Sheetfile" "MCU.kicad_sch"
-			(at 35.56 51.3846 0)
+			(at 69.85 69.1646 0)
 			(show_name no)
 			(do_not_autoplace no)
@@
 		)
 		(property "Field2" ""
-			(at 35.56 29.21 0)
+			(at 69.85 35.56 0)
 			(hide yes)
 			(show_name no)
@@
 				)
 			)
+		)
+	)
+	(sheet
+		(at 43.18 55.88)
+		(size 19.05 15.24)
+		(exclude_from_sim no)
+		(in_bom yes)
+		(on_board yes)
+		(dnp no)
+		(fields_autoplaced yes)
+		(stroke
+			(width 0.1524)
+			(type solid)
+		)
+		(fill
+			(color 0 0 0 0)
+		)
+		(property "Sheetname" "CH3,4"
+			(at 43.18 55.1684 0)
+			(show_name no)
+			(do_not_autoplace no)
+			(effects
+				(font
+					(size 1.27 1.27)
+				)
+				(justify left bottom)
+			)
+		)
+		(property "Sheetfile" "CH3,4.kicad_sch"
+			(at 43.18 71.7046 0)
+			(show_name no)
+			(do_not_autoplace no)
+			(effects
+				(font
+					(size 1.27 1.27)
+				)
+				(justify left top)
+			)
+		)
+		(instances
+			(project "E4"
+				(path "/7664cc8d-15c4-46a0-b3f4-8b4373008b19"
+					(page "5")
+				)
+			)
